File: Teensy36 CAN Bus.sch (EAGLE design)
At the start: 42 parts, among them J1 CONN_34PIN_VERT, J2 CONN_34PIN_VERT, J3 SOLDER_POINT, J4 SOLDER_POINT, J5 SOLDER_POINT, J6 SOLDER_POINT, J7 SOLDER_POINT, J8 SOLDER_POINT, U1 SN65HVD230DR, U2 SN65HVD230DR

Commit message: Update Teensy pinout
Parts:
- added R21, R22: 0Ω, AlphaLibrary:RESISTOR
- J1, J2: value CONN_34PIN_VERT -> CONN_24PIN_VERT; device AlphaLibrary:CONN_34PIN_VERT -> AlphaLibrary:CONN_24PIN_VERT
Connections:
- net 3V3: now also J2.15; no longer J2.25
- net 5V0: now also R21.2, R22.2
- net CAN1_RX: now also J1.23; no longer J1.33
- net CAN1_TX: now also J1.24; no longer J1.34
- net GND: now also J1.15; no longer J1.25
- net STBY0: now also J2.11; no longer J2.17
- net STBY1: now also J1.7; no longer J1.17
- net VIO0: now also R21.1
- net VIO1: now also R22.1
